File: KICAD_STM32.kicad_pcb (KiCad board)
At the start: 2 copper layers, 79.6 x 87.2 mm, 22 parts, among them J1 Conn_01x03_Socket, J2 Conn_01x03_Socket, J3 Screw_Terminal_01x03, SW1 SW_Push, SW2 SW_Push, SW3 SW_Push

Commit message: fixed errors in the board trace
Routing:
- net Pot1: track 42.5 -> 45.8 mm
Other:
- outline, holes or cut-outs redrawn
Changed lines of the file:
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@@
     )
   )
-  (gr_rect (start 162.1155 99.086) (end 194.5005 47.27)
+  (gr_rect (start 162.1155 47.27) (end 194.5005 99.086)
     (stroke (width 0.15) (type default)) (fill none) (layer "B.SilkS"))
-  (gr_rect (start 185.7375 85.497) (end 192.7225 63.78)
+  (gr_rect (start 185.7375 63.78) (end 192.7225 85.497)
     (stroke (width 0.15) (type default)) (fill none) (layer "B.SilkS"))
   (gr_circle (center 178.308 73.178) (end 177.1835 73.1975)
@@
     (stroke (width 0.1) (type default)) (fill none) (layer "Edge.Cuts"))
   (gr_circle (center 122.3772 124.6632) (end 122.3772 123.1392)
+    (stroke (width 0.1) (type default)) (fill none) (layer "Edge.Cuts"))
+  (gr_rect (start 185.7248 63.7032) (end 192.7352 85.4456)
     (stroke (width 0.1) (type default)) (fill none) (layer "Edge.Cuts"))
   (dimension (type aligned) (layer "B.SilkS")
@@
   (segment (start 153.797 54.61) (end 153.797 84.8106) (width 0.7) (layer "F.Cu") (net 11))
   (segment (start 185.319 52.985) (end 182.753 52.985) (width 0.7) (layer "F.Cu") (net 38))
-  (segment (start 191.1985 90.456) (end 191.1985 58.8645) (width 0.7) (layer "F.Cu") (net 38))
-  (segment (start 191.1985 58.8645) (end 185.319 52.985) (width 0.7) (layer "F.Cu") (net 38))
-  (segment (start 188.6585 90.456) (end 188.6585 63.9445) (width 0.7) (layer "F.Cu") (net 39))
+  (segment (start 191.1985 90.456) (end 195.1736 86.4809) (width 0.7) (layer "F.Cu") (net 38))
+  (segment (start 195.1736 86.4809) (end 195.1736 62.8396) (width 0.7) (layer "F.Cu") (net 38))
+  (segment (start 195.1736 62.8396) (end 185.319 52.985) (width 0.7) (layer "F.Cu") (net 38))
+  (segment (start 183.9976 85.7951) (end 183.9976 59.2836) (width 0.7) (layer "F.Cu") (net 39))
+  (segment (start 183.9976 59.2836) (end 177.699 52.985) (width 0.7) (layer "F.Cu") (net 39))
+  (segment (start 188.6585 90.456) (end 183.9976 85.7951) (width 0.7) (layer "F.Cu") (net 39))
   (segment (start 177.699 52.985) (end 175.26 52.985) (width 0.7) (layer "F.Cu") (net 39))
-  (segment (start 188.6585 63.9445) (end 177.699 52.985) (width 0.7) (layer "F.Cu") (net 39))
-  (segment (start 163.6982 55.9308) (end 155.321 64.308) (width 0.7) (layer "F.Cu") (net 40))
-  (segment (start 186.1185 63.8937) (end 178.1556 55.9308) (width 0.7) (layer "F.Cu") (net 40))
+  (segment (start 181.9148 86.2523) (end 181.9148 59.69) (width 0.7) (layer "F.Cu") (net 40))
   (segment (start 178.1556 55.9308) (end 163.6982 55.9308) (width 0.7) (layer "F.Cu") (net 40))
   (segment (start 155.321 85.8266) (end 147.828 93.3196) (width 0.7) (layer "F.Cu") (net 40))
+  (segment (start 186.1185 90.456) (end 181.9148 86.2523) (width 0.7) (layer "F.Cu") (net 40))
+  (segment (start 181.9148 59.69) (end 178.1556 55.9308) (width 0.7) (layer "F.Cu") (net 40))
+  (segment (start 163.6982 55.9308) (end 155.321 64.308) (width 0.7) (layer "F.Cu") (net 40))
   (segment (start 155.321 64.308) (end 155.321 85.8266) (width 0.7) (layer "F.Cu") (net 40))
-  (segment (start 186.1185 90.456) (end 186.1185 63.8937) (width 0.7) (layer "F.Cu") (net 40))
   (zone (net 1) (net_name "GND") (layer "F.Cu") (hatch edge 0.5)
     (connect_pads (clearance 0.5))

Commit message: add new resistor
Parts:
- added R8: R, Resistor_SMD:R_1206_3216Metric_Pad1.30x1.75mm_HandSolder, F.Cu at (151.9, 64.2)
- added R9: R, Resistor_SMD:R_1206_3216Metric_Pad1.30x1.75mm_HandSolder, F.Cu at (153.9, 58.1)
Connections:
- C7 pad 1: -5V -> GND
- C7 pad 2: GND -> -5V
- R4 pad 2: ADC0 -> Net-(R4-Pad2)
- R5 pad 2: ADC0 -> Net-(R4-Pad2)
- R6 pad 2: ADC1 -> Net-(R6-Pad2)
- R7 pad 2: ADC1 -> Net-(R6-Pad2)
Routing:
- net ADC0: track 93.8 -> 24.2 mm
- net Net-(R4-Pad2): track 0.00 -> 66.5 mm
- net ADC1: track 67.9 -> 33.6 mm
- net Net-(R6-Pad2): track 0.00 -> 31.2 mm
