File: KICAD_STM32.kicad_sch (KiCad schematic)
At the start: 22 parts, among them J1 Conn_01x03_Socket, J2 Conn_01x03_Socket, J3 Screw_Terminal_01x03, SW1 SW_Push, SW2 SW_Push, SW3 SW_Push

Commit message: add new resistor
Parts:
- added R8, R9: R, Resistor_SMD:R_1206_3216Metric_Pad1.30x1.75mm_HandSolder, symbol Device:R
Connections:
- net ADC0: now also R8.2; no longer R4.2, R5.2
- net ADC1: now also R9.1; no longer R6.2, R7.2
- new net: R4.2, R5.2, R8.1
- new net: R6.2, R7.2, R9.2
Changed lines of the file:
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@@
   (junction (at 58.42 78.74) (diameter 0) (color 0 0 0 0)
   )
+  (junction (at 93.98 123.19) (diameter 0) (color 0 0 0 0)
+  )
   (junction (at 223.52 111.76) (diameter 0) (color 0 0 0 0)
   )
+  (junction (at 107.95 123.19) (diameter 0) (color 0 0 0 0)
+  )
   (junction (at 59.69 59.69) (diameter 0) (color 0 0 0 0)
   )
@@
     (stroke (width 0) (type default))
   )
+  (wire (pts (xy 107.95 121.92) (xy 107.95 123.19))
+    (stroke (width 0) (type default))
+  )
+  (wire (pts (xy 91.44 123.19) (xy 93.98 123.19))
+    (stroke (width 0) (type default))
+  )
   (wire (pts (xy 48.26 59.69) (xy 48.26 67.31))
     (stroke (width 0) (type default))
@@
     (stroke (width 0) (type default))
   )
+  (wire (pts (xy 82.55 123.19) (xy 83.82 123.19))
+    (stroke (width 0) (type default))
+  )
   (wire (pts (xy 223.52 140.97) (xy 223.52 148.59))
     (stroke (width 0) (type default))
@@
     (stroke (width 0) (type default))
   )
+  (wire (pts (xy 119.38 123.19) (xy 118.11 123.19))
+    (stroke (width 0) (type default))
+  )
   (wire (pts (xy 135.89 105.41) (xy 143.51 105.41))
     (stroke (width 0) (type default))
@@
     (stroke (width 0) (type default))
   )
+  (wire (pts (xy 110.49 123.19) (xy 107.95 123.19))
+    (stroke (width 0) (type default))
+  )
   (wire (pts (xy 48.26 86.36) (xy 48.26 78.74))
     (stroke (width 0) (type default))
@@
     (stroke (width 0) (type default))
   )
+  (wire (pts (xy 138.43 115.57) (xy 143.51 115.57))
+    (stroke (width 0) (type default))
+  )
+  (wire (pts (xy 59.69 50.8) (xy 59.69 59.69))
+    (stroke (width 0) (type default))
+  )
+  (wire (pts (xy 173.99 97.79) (xy 194.31 97.79))
+    (stroke (width 0) (type default))
+  )
+  (wire (pts (xy 49.53 86.36) (xy 48.26 86.36))
+    (stroke (width 0) (type default))
+  )
+  (wire (pts (xy 223.52 111.76) (xy 223.52 119.38))
+    (stroke (width 0) (type default))
+  )
   (wire (pts (xy 93.98 121.92) (xy 93.98 123.19))
     (stroke (width 0) (type default))
   )
-  (wire (pts (xy 138.43 115.57) (xy 143.51 115.57))
-    (stroke (width 0) (type default))
-  )
-  (wire (pts (xy 59.69 50.8) (xy 59.69 59.69))
-    (stroke (width 0) (type default))
-  )
-  (wire (pts (xy 173.99 97.79) (xy 194.31 97.79))
-    (stroke (width 0) (type default))
-  )
-  (wire (pts (xy 107.95 121.92) (xy 107.95 123.19))
-    (stroke (width 0) (type default))
-  )
-  (wire (pts (xy 49.53 86.36) (xy 48.26 86.36))
-    (stroke (width 0) (type default))
-  )
-  (wire (pts (xy 223.52 111.76) (xy 223.52 119.38))
-    (stroke (width 0) (type default))
-  )
   (wire (pts (xy 154.94 69.85) (xy 154.94 77.47))
     (stroke (width 0) (type default))
@@
     )
   )
-  (global_label "ADC0" (shape output) (at 93.98 123.19 180) (fields_autoplaced)
-    (effects (font (size 1.27 1.27)) (justify right))
-    (property "Intersheetrefs" "${INTERSHEET_REFS}" (at 86.2361 123.19 0)
+  (global_label "ADC0" (shape output) (at 82.55 123.19 180) (fields_autoplaced)
+    (effects (font (size 1.27 1.27)) (justify right))
+    (property "Intersheetrefs" "${INTERSHEET_REFS}" (at 74.8061 123.19 0)
       (effects (font (size 1.27 1.27)) (justify right) hide)
     )
@@
     )
   )
-  (global_label "ADC1" (shape output) (at 107.95 123.19 0) (fields_autoplaced)
-    (effects (font (size 1.27 1.27)) (justify left))
-    (property "Intersheetrefs" "${INTERSHEET_REFS}" (at 115.6939 123.19 0)
+  (global_label "ADC1" (shape output) (at 119.38 123.19 0) (fields_autoplaced)
+    (effects (font (size 1.27 1.27)) (justify left))
+    (property "Intersheetrefs" "${INTERSHEET_REFS}" (at 127.1239 123.19 0)
       (effects (font (size 1.27 1.27)) (justify left) hide)
     )
@@
     )
   )
+  (symbol (lib_id "Device:R") (at 87.63 123.19 270) (unit 1)
+    (in_bom yes) (on_board yes) (dnp no) (fields_autoplaced)
+    (property "Reference" "R8" (at 87.63 118.11 90)
+      (effects (font (size 1.27 1.27)))
+    )
+    (property "Value" "R" (at 87.63 120.65 90)
+      (effects (font (size 1.27 1.27)))
+    )
+    (property "Footprint" "Resistor_SMD:R_1206_3216Metric_Pad1.30x1.75mm_HandSolder" (at 87.63 121.412 90)
+      (effects (font (size 1.27 1.27)) hide)
+    )
+    (property "Datasheet" "~" (at 87.63 123.19 0)
+      (effects (font (size 1.27 1.27)) hide)
+    )
+    (pin "1")
+    (pin "2")
+    (instances
+      (project "KICAD_STM32"
+        (path "/9adf92ad-bf22-4193-ab21-9dbe2888d011"
+          (reference "R8") (unit 1)
+        )
+      )
+    )
+  )
   (symbol (lib_id "power:-5V") (at 224.79 77.47 180) (unit 1)
     (in_bom yes) (on_board yes) (dnp no) (fields_autoplaced)
@@
         )
       )
+    )
+  )
+  (symbol (lib_id "Device:R") (at 114.3 123.19 270) (unit 1)
+    (in_bom yes) (on_board yes) (dnp no) (fields_autoplaced)
+    (property "Reference" "R9" (at 114.3 118.11 90)
+      (effects (font (size 1.27 1.27)))
+    )
+    (property "Value" "R" (at 114.3 120.65 90)
+      (effects (font (size 1.27 1.27)))
+    )
+    (property "Footprint" "Resistor_SMD:R_1206_3216Metric_Pad1.30x1.75mm_HandSolder" (at 114.3 121.412 90)
+      (effects (font (size 1.27 1.27)) hide)
+    )
+    (property "Datasheet" "~" (at 114.3 123.19 0)
+      (effects (font (size 1.27 1.27)) hide)
+    )
+    (pin "1")
+    (pin "2")
+    (instances
+      (project "KICAD_STM32"
+        (path "/9adf92ad-bf22-4193-ab21-9dbe2888d011"
+          (reference "R9") (unit 1)
+        )
+      )
